File: Buck_Converter/Buck_ConverterV1/Buck_ConverterV1.kicad_pcb (KiCad board)
At the start: 2 copper layers, 11 parts, among them J1 Screw_Terminal_01x02, J2 Screw_Terminal_01x02, U1 LTC3624EDD-PBF

Commit message: footprint and layout change base
Parts:
- U1: footprint LTC3624:DFN-8_DD_LIT -> Package_DFN_QFN:DFN-8-1EP_3x3mm_P0.5mm_EP1.66x2.38mm
- moved C1 36.9 mm to (121.3, 100.5), turned to -90 degrees
- moved J1 31.7 mm to (111.7, 98.0), turned to -90 degrees
- moved U1 30.9 mm to (130.0, 100.0)
- moved L1 30.0 mm to (130.1, 94.1)
- moved C2 28.5 mm to (126.4, 101.5), turned to -90 degrees
- moved C3 28.4 mm to (133.4, 99.3), turned to 90 degrees
- moved C4 24.2 mm to (135.0, 95.1), turned to -90 degrees
- moved R3 23.8 mm to (130.4, 106.3), turned to 180 degrees
- moved R1 20.6 mm to (134.1, 102.4), turned to 180 degrees
- moved R2 20.4 mm to (134.1, 104.5)
- moved J2 2.98 mm to (142.7, 102.4), turned to 90 degrees
Routing:
- net GND: vias 0 -> 6
- added copper zone on B.Cu, net GND
Other:
- board outline added: 41.8 x 18.3 mm
- board text added: "+ VIN 9-15V"
- board text added: "+5V OUT"
- board text added: "GND"
- board text added: "LTC3624 BUCK V1"
