File: Buck_Converter/Buck_ConverterV1/Buck_ConverterV1.kicad_sch (KiCad schematic)
At the start: 11 parts, among them J1 Screw_Terminal_01x02, J2 Screw_Terminal_01x02, U1 LTC3624EDD-PBF

Commit message: footprint and layout change base
Parts:
- U1: footprint LTC3624:DFN-8_DD_LIT -> Package_DFN_QFN:DFN-8-1EP_3x3mm_P0.5mm_EP1.66x2.38mm
Changed lines of the file:
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@@
 			)
 		)
-		(property "Footprint" "LTC3624:DFN-8_DD_LIT"
+		(property "Footprint" "Package_DFN_QFN:DFN-8-1EP_3x3mm_P0.5mm_EP1.66x2.38mm"
 			(at 116.84 90.17 0)
 			(hide yes)
